File: Hardware/Kicad File/OpenWear.kicad_pcb (KiCad board)
At the start: 4 copper layers, 50 x 50 mm, 41 parts, among them J1 USB_C, J2 Connector, Q1 BC847B, Q2 DMG3415U, U1 ESP32-PICO-D4, U2 BMP280, U3 CH343P, U4 TLV70233_SOT23-5, U5 MCP73831-2-OT, U6 LSM6DS3

Commit message: update kicad
Parts:
- D1: value Inolux_IN-PI554FCH -> XL-5050RGBC-WS2812B
- E1: value Antenna -> ANT_CA-C03
- Q1: value BC847B -> BC847BS
- S1, S2: value TL3365AF180QG -> UK-B0267-SP25Y
- U4: value TLV70233_SOT23-5 -> ME6211C33M5G-N
- U5: value MCP73831-2-OT -> MCP73831T-2ATI/OT
- U6: value LSM6DS3 -> LSM6DS3TR
- moved C1 42.7 mm to (193.3, 99.3)
- moved U4 42.7 mm to (195.9, 99.3)
- moved C2 42.7 mm to (198.6, 99.2)
- moved Q2 42.6 mm to (195.6, 71.8), turned to -90 degrees
- moved Q1 42.5 mm to (199.9, 84.3)
- moved R3 42.5 mm to (197.3, 84.3)
- moved R4 42.5 mm to (202.5, 84.3)
- moved C5 40.7 mm to (193.4, 78.2)
- moved U3 40.7 mm to (190.4, 78.2)
- moved C4 40.7 mm to (187.2, 78.4), turned to -90 degrees
- moved C9 30.1 mm to (106.3, 100.2)
- moved U2 30.1 mm to (109.0, 100.0)
- moved C7 30.1 mm to (109.0, 102.6)
- moved U5 26.9 mm to (188.6, 71.8), turned to 90 degrees
- moved C3 25.8 mm to (192.9, 72.0), turned to -90 degrees
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Routing:
- net /D+: track 22.6 -> 5.22 mm, vias 2 -> 1
- net /D-: track 19.0 -> 2.52 mm, vias 3 -> 2
- net /EN: track 5.52 -> 0.00 mm
- net VCC: track 4.72 -> 0.00 mm
- net VBUS: track 16.6 -> 13.9 mm
- net /TX: track 1.92 -> 0.00 mm, vias 1 -> 0
- net +3V3: track 1.63 -> 0.00 mm, vias 3 -> 0
- net /RX: track 1.15 -> 0.00 mm, vias 1 -> 0

Commit message: update pcb
Parts:
- moved C9 79.3 mm to (185.6, 102.4), turned to 0 degrees
- moved U2 76.7 mm to (185.6, 104.7)
- moved C7 76.7 mm to (185.6, 107.0), turned to 180 degrees
- moved Q2 51.7 mm to (144.3, 78.3), turned to 90 degrees
- moved A1 43.8 mm to (200.2, 110.6)
- moved R6 43.8 mm to (200.2, 112.1)
- moved U6 28.0 mm to (185.6, 109.8)
- moved C8 28.0 mm to (188.3, 109.6)

Commit message: update kicad
Parts:
- removed R10, R9: 0, Resistor_SMD:R_0603_1608Metric
- moved C9 49.2 mm to (136.8, 95.8), turned to 90 degrees
- moved U2 47.3 mm to (139.1, 95.9), turned to 90 degrees
- moved R6 43.9 mm to (157.6, 101.4)
- moved A1 43.8 mm to (157.6, 99.9)
- moved C8 33.3 mm to (157.6, 96.7), turned to 180 degrees
- moved C7 30.4 mm to (157.6, 95.1)
- moved U6 28.1 mm to (161.0, 96.1), turned to -90 degrees
- moved C2 21.6 mm to (214.4, 84.6)
- moved C1 21.6 mm to (209.1, 84.6)
- moved U4 21.6 mm to (211.7, 84.6)
- moved R5 7.27 mm to (140.9, 83.2)
- moved C6 7.27 mm to (142.5, 83.3)
- moved R7 3.81 mm to (142.4, 96.7)
- moved R8 3.79 mm to (142.4, 98.4)
- moved C10 0.20 mm to (157.6, 98.4)
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Connections:
- R7 pad 1: /SCL -> /IO22_SCL
- R8 pad 1: /SDA -> /IO21_SDA
- U1 pad 39: /IO22 -> /IO22_SCL
- U1 pad 42: /IO21 -> /IO21_SDA
- U2 pad 3: /SDA -> /IO21_SDA
- U2 pad 4: /SCL -> /IO22_SCL
- U6 pad 13: /SCL -> /IO22_SCL
- U6 pad 14: /SDA -> /IO21_SDA
Other:
- board text added: "3V3"
- board text added: "5V"
- board text added: "A0"
- board text added: "A1"
- board text added: "A10"
- board text added: "A2"
- board text added: "A3"
- board text added: "A4"
- board text added: "A5"
- board text added: "A6"
- board text added: "A7"
- board text added: "A8"
- board text added: "A9"
- board text added: "GND"
