File: Hardware/Kicad File/OpenWear.kicad_pcb (KiCad board)
At the start: 4 copper layers, 50 x 50 mm, 39 parts, among them J1 USB_C, J2 Connector, Q1 BC847BS, Q2 DMG3415U, U1 ESP32-PICO-D4, U2 BMP280, U3 CH343P, U4 ME6211C33M5G-N, U5 MCP73831T-2ATI/OT, U6 LSM6DS3TR

Commit message: update pcb
Routing:
- net +3V3: track 0.00 -> 14.1 mm
- net /IO21_SDA: track 0.00 -> 6.00 mm, vias 0 -> 2
- net /IO22_SCL: track 0.00 -> 5.05 mm, vias 0 -> 2
- net /TX: track 0.00 -> 2.23 mm, vias 0 -> 1
- net /RX: track 0.00 -> 1.52 mm, vias 0 -> 1
- added copper zone on In2.Cu, net +3V3
- removed copper zone on In2.Cu, net GND
Changed lines of the file:
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@@
   (via (at 149.746 71.9152) (size 0.5) (drill 0.3) (layers "F.Cu" "B.Cu") (net 5))
   (via (at 150.763 71.9152) (size 0.5) (drill 0.3) (layers "F.Cu" "B.Cu") (net 5))
+  (segment (start 145.75 98.6054) (end 144.25 100.1054) (width 0.25) (layer "F.Cu") (net 8))
+  (segment (start 143.155 100.033) (end 143.2274 100.1054) (width 0.25) (layer "F.Cu") (net 8))
+  (segment (start 143.2764 101.8054) (end 143.155 101.684) (width 0.25) (layer "F.Cu") (net 8))
+  (segment (start 146.55 95.6054) (end 143.6804 95.6054) (width 0.25) (layer "F.Cu") (net 8))
+  (segment (start 144.25 100.1054) (end 146.55 100.1054) (width 0.25) (layer "F.Cu") (net 8))
+  (segment (start 146.55 98.6054) (end 145.75 98.6054) (width 0.25) (layer "F.Cu") (net 8))
+  (segment (start 143.2274 100.1054) (end 144.25 100.1054) (width 0.25) (layer "F.Cu") (net 8))
+  (segment (start 147.25 101.8054) (end 143.2764 101.8054) (width 0.25) (layer "F.Cu") (net 8))
+  (segment (start 143.6804 95.6054) (end 143.155 95.08) (width 0.25) (layer "F.Cu") (net 8))
   (segment (start 147.75 110.672) (end 147.4416 110.9804) (width 0.25) (layer "F.Cu") (net 9))
   (segment (start 147.75 101.8054) (end 147.75 110.672) (width 0.25) (layer "F.Cu") (net 9))
@@
   (segment (start 152.45 88.4) (end 151.3968 88.4) (width 0.127) (layer "F.Cu") (net 11))
   (segment (start 150.75 89.0468) (end 150.75 94.9054) (width 0.127) (layer "F.Cu") (net 11))
+  (segment (start 142.4045 96.744416) (end 143.191584 96.744416) (width 0.127) (layer "F.Cu") (net 41))
+  (segment (start 139.1542 94.9276) (end 139.1444 94.9178) (width 0.127) (layer "F.Cu") (net 41))
+  (segment (start 143.3306 96.6054) (end 146.55 96.6054) (width 0.127) (layer "F.Cu") (net 41))
+  (segment (start 143.191584 96.744416) (end 143.3306 96.6054) (width 0.25) (layer "F.Cu") (net 41))
+  (segment (start 143.191584 96.744416) (end 143.205 96.731) (width 0.127) (layer "F.Cu") (net 41))
+  (segment (start 139.1444 94.9178) (end 138.3288 94.9178) (width 0.127) (layer "F.Cu") (net 41))
+  (via (at 142.4045 96.744416) (size 0.5) (drill 0.3) (layers "F.Cu" "B.Cu") (net 41))
+  (via (at 139.1542 94.9276) (size 0.5) (drill 0.3) (layers "F.Cu" "B.Cu") (net 41))
+  (segment (start 138.8038 95.5678) (end 138.3288 95.5678) (width 0.127) (layer "F.Cu") (net 42))
+  (segment (start 145.5522 98.1054) (end 146.55 98.1054) (width 0.127) (layer "F.Cu") (net 42))
+  (segment (start 142.4045 98.382) (end 145.2756 98.382) (width 0.127) (layer "F.Cu") (net 42))
+  (segment (start 145.2756 98.382) (end 145.5522 98.1054) (width 0.127) (layer "F.Cu") (net 42))
+  (segment (start 142.4045 98.382) (end 143.205 98.382) (width 0.127) (layer "F.Cu") (net 42))
+  (segment (start 139.1288 95.8928) (end 138.8038 95.5678) (width 0.127) (layer "F.Cu") (net 42))
+  (via (at 139.1288 95.8928) (size 0.5) (drill 0.3) (layers "F.Cu" "B.Cu") (net 42))
+  (via (at 142.4045 98.382) (size 0.5) (drill 0.3) (layers "F.Cu" "B.Cu") (net 42))
   (segment (start 148.5778 88.4) (end 147.55 88.4) (width 0.25) (layer "F.Cu") (net 54))
   (segment (start 148.25 93.655) (end 149.0602 92.8448) (width 0.25) (layer "F.Cu") (net 54))
@@
   (segment (start 148.25 94.9054) (end 148.25 93.655) (width 0.25) (layer "F.Cu") (net 54))
   (segment (start 149.0602 88.8824) (end 148.5778 88.4) (width 0.25) (layer "F.Cu") (net 54))
-  (zone (net 1) (net_name "GND") (layers "F.Cu" "In1.Cu" "In2.Cu" "B.Cu") (hatch edge 0.5)
-    (connect_pads (clearance 0))
-    (min_thickness 0.25) (filled_areas_thickness no)
-    (fill yes (thermal_gap 0.3) (thermal_bridge_width 0.3) (smoothing fillet) (radius 0.1))
-    (polygon
-      (pts
-        (xy 120 60)
-        (xy 180 60)
-        (xy 180 120)
-        (xy 120 120)
-      )
-    )
-  )
+  (segment (start 146.55 97.1054) (end 144.7234 97.1054) (width 0.127) (layer "F.Cu") (net 61))
+  (segment (start 146.5434 97.112) (end 146.55 97.1054) (width 0.127) (layer "F.Cu") (net 61))
+  (segment (start 144.7234 97.1054) (end 144.4628 97.366) (width 0.127) (layer "F.Cu") (net 61))
+  (segment (start 144.4628 97.366) (end 144.4882 97.366) (width 0.127) (layer "F.Cu") (net 61))
+  (via (at 144.4628 97.366) (size 0.5) (drill 0.3) (layers "F.Cu" "B.Cu") (net 61))
+  (segment (start 145.116054 97.816054) (end 145.326708 97.6054) (width 0.127) (layer "F.Cu") (net 62))
+  (segment (start 145.326708 97.6054) (end 146.55 97.6054) (width 0.127) (layer "F.Cu") (net 62))
+  (via (at 145.116054 97.816054) (size 0.5) (drill 0.3) (layers "F.Cu" "B.Cu") (net 62))
   (zone (net 0) (net_name "") (layers "F.Cu" "In1.Cu" "In2.Cu" "B.Cu") (hatch full 0.5)
     (connect_pads (clearance 0))
@@
       )
     )
+  )
+  (zone (net 1) (net_name "GND") (layers "F.Cu" "In1.Cu" "B.Cu") (hatch edge 0.5)
+    (connect_pads (clearance 0))
+    (min_thickness 0.25) (filled_areas_thickness no)
+    (fill yes (thermal_gap 0.3) (thermal_bridge_width 0.3) (smoothing fillet) (radius 0.1))
+    (polygon
+      (pts
+        (xy 120 60)
+        (xy 180 60)
+        (xy 180 120)
+        (xy 120 120)
+      )
+    )
+  )
+  (zone (net 8) (net_name "+3V3") (layer "In2.Cu") (hatch edge 0.5)
+    (priority 1)
+    (connect_pads (clearance 0))
+    (min_thickness 0.25) (filled_areas_thickness no)
+    (fill yes (thermal_gap 0.3) (thermal_bridge_width 0.3) (smoothing fillet) (radius 0.1))
+    (polygon
+      (pts
+        (xy 175.4 64.6)
+        (xy 175.4 115.4)
+        (xy 124.6 115.4)
+        (xy 124.6 64.6)
+      )
+    )

Commit message: update PCB layout
Parts:
- added REF**: Pin_D1.0mm_L10.0mm, Connector_Pin:Pin_D1.0mm_L10.0mm, F.Cu at (157.0, 68.5)
- added REF**: Pin_D1.0mm_L10.0mm, Connector_Pin:Pin_D1.0mm_L10.0mm, F.Cu at (143.0, 68.5)
- moved R4 51.8 mm to (150.8, 83.7)
- moved Q1 45.2 mm to (154.7, 83.7)
- moved R3 45.0 mm to (152.3, 83.7)
- moved C5 44.5 mm to (149.2, 83.7)
- moved U3 44.5 mm to (146.2, 83.6)
- moved C4 44.2 mm to (143.3, 83.8)
- moved D3 20.2 mm to (175.1, 54.8)
- moved U5 20.2 mm to (177.8, 54.8)
- moved R2 20.2 mm to (180.5, 54.9)
- moved R1 20.2 mm to (173.5, 54.8)
- moved C3 20.2 mm to (182.1, 54.9)
- moved R5 1.03 mm to (140.0, 83.7)
- moved C6 1.01 mm to (141.6, 83.8)

Commit message: update pcb and sch
Parts:
- added C15: 4.7uF, Capacitor_SMD:C_0603_1608Metric, F.Cu at (153.7, 78.3)
- C3: value 100nF -> 4.7uF
- R1: value 10K -> 1K
- moved C1 62.9 mm to (146.5, 78.3)
- moved U4 62.8 mm to (149.2, 78.3)
- moved C2 62.8 mm to (151.9, 78.3)
- moved C3 37.9 mm to (157.3, 83.6)
- moved R2 35.9 mm to (159.0, 83.6)
- moved U5 31.8 mm to (156.4, 78.3), turned to -90 degrees
- moved R1 31.5 mm to (160.7, 83.6)
- moved D3 28.4 mm to (159.1, 78.3), turned to -90 degrees
- moved R5 0.64 mm to (139.3, 83.6)
- moved C6 0.61 mm to (141.0, 83.6)
- moved C4 0.58 mm to (142.7, 83.6)
- moved Q2 0.47 mm to (143.8, 78.3)
- moved U3 0.44 mm to (145.8, 83.6)
- moved C5 0.42 mm to (148.8, 83.6)
- moved D2 0.36 mm to (140.9, 78.3)
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Connections:
- C3 pad 1: GND -> +5V
- C3 pad 2: +BATT -> GND
- J2 pad 14: VCC -> +5V
- R2 pad 1: +BATT -> GND
- R5 pad 1: +3.3V -> +3V3
- U3 pad 12: unconnected-(U3-DTR-Pad12) -> /DTR
- U3 pad 13: unconnected-(U3-RTS-Pad13) -> /RTS
Routing:
- net +3V3: track 14.1 -> 57.6 mm, vias 0 -> 9
- net +5V: track 0.00 -> 40.5 mm, vias 0 -> 3
- net +BATT: track 0.00 -> 24.6 mm
- net /EN: track 0.00 -> 21.2 mm, vias 0 -> 2
- net /D+: track 5.22 -> 23.1 mm, vias 1 -> 2
- net /D-: track 2.52 -> 19.2 mm, vias 2 -> 3
- net /RTS: track 0.00 -> 15.8 mm, vias 0 -> 2
- net /TX: track 2.23 -> 15.5 mm, vias 1 -> 2
- net /RX: track 1.52 -> 14.4 mm, vias 1 -> 2
- net /IO0: track 0.00 -> 12.1 mm
- net VCC: track 0.00 -> 8.23 mm
- net /DTR: track 0.00 -> 8.07 mm
- net Net-(Q1A-B1): track 0.00 -> 5.28 mm
- net Net-(D3-A): track 0.00 -> 4.77 mm
- net Net-(U5-PROG): track 0.00 -> 4.56 mm
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- added copper zone on F.Cu, net +3V3
Other:
- board text removed: "3V3"
- board text removed: "5V"
- board text removed: "A0"
- board text removed: "A1"
- board text removed: "A10"
- board text removed: "A3"
- board text removed: "A4"
- board text removed: "A5"
- board text removed: "A6"
- board text removed: "A7"
- board text removed: "A8"
- board text removed: "A9"
- board text removed: "GND"

Commit message: update pcb layout
Routing:
- net /IO22_SCL: track 1.83 -> 33.1 mm, vias 2 -> 3
- net /IO21_SDA: track 6.00 -> 33.5 mm, vias 2 -> 3
- net /SCL1: track 0.00 -> 22.4 mm
- net /IO13: track 0.00 -> 21.7 mm, vias 0 -> 1
- net /SDA1: track 0.00 -> 20.4 mm
- net /IO12: track 0.00 -> 17.7 mm, vias 0 -> 1
- net /IO14: track 0.00 -> 17.6 mm
- net /IO27: track 0.00 -> 13.5 mm
- net NEOPIXEL_I2C_POWER: track 8.07 -> 21.0 mm, vias 0 -> 2
- net +3V3: track 57.6 -> 49.1 mm, vias 9 -> 11
- net /D-: track 19.2 -> 20.2 mm
- net +5V: track 40.5 -> 39.7 mm, vias 3 -> 2
- net GND: track 1.86 -> 1.03 mm
- net /D+: track 23.1 -> 23.9 mm
- net /RTS: track 15.8 -> 15.2 mm
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
Commit message: update pcb layout
Parts:
- moved E1 0.86 mm to (150.1, 111.8)
Routing:
- net /IO21_SDA: track 33.5 -> 3.46 mm, vias 3 -> 0
- net /IO22_SCL: track 33.1 -> 3.22 mm, vias 3 -> 0
- net /IO15: track 0.00 -> 29.0 mm
- net /IO13: track 21.7 -> 0.00 mm, vias 1 -> 0
- net /IO12: track 17.7 -> 2.47 mm
- net NEOPIXEL_I2C_POWER: track 21.0 -> 9.72 mm, vias 2 -> 0
- net /IO0: track 12.1 -> 21.0 mm
- net +3V3: track 49.1 -> 44.6 mm, vias 11 -> 7
- net +5V: track 39.7 -> 41.5 mm, vias 2 -> 0
- net LIGHT_SENSOR: track 0.00 -> 1.84 mm, vias 0 -> 1
- net /IO25: track 0.00 -> 1.48 mm, vias 0 -> 1
- net /IO26: track 0.00 -> 1.39 mm, vias 0 -> 1
- net /EN: track 21.7 -> 23.1 mm, vias 2 -> 3
- net Net-(U1-LNA_IN): track 8.87 -> 10.2 mm
- net /IO4: track 0.00 -> 1.26 mm, vias 0 -> 1
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
Commit message: update pcb and sch
Parts:
- added C16: 100nF, Capacitor_SMD:C_0603_1608Metric, F.Cu at (139.0, 98.8)
- moved C9 0.49 mm to (136.5, 96.2)
- moved U2 0.42 mm to (139.0, 96.3)
- moved U1 0.41 mm to (150.0, 98.8)
- moved C11 0.39 mm to (150.0, 104.1)
- moved C8 0.39 mm to (157.6, 97.1)
- moved R7 0.39 mm to (142.4, 97.1)
- moved A1 0.39 mm to (157.6, 100.3)
- moved C10 0.39 mm to (157.6, 98.8)
- moved C12 0.39 mm to (142.4, 100.4)
- moved C13 0.39 mm to (142.4, 102.1)
- moved R6 0.39 mm to (157.6, 101.8)
- moved U6 0.39 mm to (161.0, 96.5)
- moved C14 0.38 mm to (142.4, 95.5)
- moved C7 0.38 mm to (157.6, 95.5)
- moved R8 0.38 mm to (142.4, 98.8)
Connections:
- U3 pad 9: unconnected-(U3-VBUS-Pad9) -> +3V3
Routing:
- net /IO4: track 1.26 -> 41.5 mm
- net /IO2: track 1.22 -> 38.6 mm
- net /IO22_SCL: track 3.22 -> 36.3 mm, vias 0 -> 5
- net /IO21_SDA: track 3.46 -> 35.6 mm, vias 0 -> 5
- net /IO26: track 1.39 -> 25.9 mm, vias 1 -> 2
- net /IO13: track 0.00 -> 22.1 mm, vias 0 -> 2
- net /EN: track 23.1 -> 42.4 mm, vias 3 -> 5
- net /IO25: track 1.48 -> 20.6 mm
- net /IO12: track 2.47 -> 17.8 mm
- net NEOPIXEL_I2C_POWER: track 9.72 -> 24.5 mm, vias 0 -> 3
- net +3V3: track 44.6 -> 54.9 mm, vias 7 -> 13
- net LIGHT_SENSOR: track 1.84 -> 10.4 mm, vias 1 -> 2
- net GND: track 1.03 -> 3.73 mm, vias 11 -> 53
- net /IO15: track 29.0 -> 29.6 mm

Commit message: update sch
Parts:
- D2: footprint Diode_SMD:D_SOD-323 -> Diode_SMD:D_SOD-323_HandSoldering
Connections:
- C3 pad 1: +5V -> VBUS
- D2 pad 1: +5V -> VCC
- J2 pad 14: +5V -> VCC
- Q2 pad 1: +5V -> VBUS
- R1 pad 2: +5V -> VBUS
- U5 pad 4: +5V -> VBUS
Routing:
- net +5V: track 41.5 -> 0.00 mm
- net VBUS: track 17.3 -> 47.3 mm
- net VCC: track 8.79 -> 36.5 mm, vias 0 -> 3
- net /IO26: track 25.9 -> 27.6 mm
- net /IO25: track 20.6 -> 22.3 mm
- net GND: vias 53 -> 102
