File: Hardware/Kicad File/OpenWear.kicad_sch (KiCad schematic)
At the start: 36 parts, among them J1 USB_C, J2 Connector, Q1 BC847B, Q2 DMG3415U, U1 ESP32-PICO-D4, U2 BMP280, U3 CH343P, U4 TLV70233_SOT23-5, U5 MCP73831-2-OT, U6 LSM6DS3

Commit message: update sch
Parts:
- added C14: 100nF, Capacitor_SMD:C_0603_1608Metric, symbol Device:C
- added R10, R9: 0, Resistor_SMD:R_0603_1608Metric, symbol Device:R
- added R7, R8: 10K, Resistor_SMD:R_0603_1608Metric, symbol Device:R
Connections:
- net +3V3: now also C14.2; no longer U1.39 (IO22), U1.42 (IO21), U2.3 (SDI), U2.4 (SCK), U6.13 (SCL), U6.14 (SDA)
- net +5V: no longer J2.14
- net D+: now also U3.7 (UD+)
- net D-: now also U3.8 (UD-)
- net GND: now also C14.1
- net IO12: now also J2.10 (A9)
- net IO13: now also J2.11 (A10)
- net IO14: now also J2.9 (A8)
- net IO15: now also J2.12 (A11)
- net IO2: now also J2.3 (A2)
- net IO25: now also J2.7 (A6)
- net IO26: now also J2.6 (A5)
- net IO27: now also J2.8 (A7)
- net IO4: now also J2.2 (A1)
- net SCL1: now also J2.4 (A3)
- net SDA1: now also J2.5 (A4)
- net VCC: now also J2.14 (5V)
- net NEOPIXEL_POWER renamed NEOPIXEL_I2C_POWER
- net NEOPIXEL_I2C_POWER: now also R7.2, R8.2
- new net IO21: R9.2, U1.42 (IO21)
- new net IO22: R10.2, U1.39 (IO22)
- new net SCL: R10.1, R7.1, U2.4 (SCK), U6.13 (SCL)
- new net SDA: R8.1, R9.1, U2.3 (SDI), U6.14 (SDA)
Other:
- moved on the sheet: C6, R5, S1, S2

Commit message: update kicad
Parts:
- A1: Availability In Stock -> (none); Check_prices https://www.snapeda.com/parts/ALS-PT19-315C/L177/TR8/Everli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 -> (none); LCSC Part # (none) -> C146233; MANUFACTURER Everlight -> (none); MAXIMUM_PACKAGE_HEIGHT 0.7 mm -> (none); MF Everlight -> (none); MP ALS-PT19-315C/L177/TR8 -> (none); PARTREV 5 -> (none); Package SMD-2 Everlight -> (none); Price None -> (none); Purchase-URL https://www.snapeda.com/api/url_track_click_mouser/?unipart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 -> (none); STANDARD Manufacturer Recommendations -> (none); SnapEDA_Link https://www.snapeda.com/parts/ALS-PT19-315C/L177/TR8/Everli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 -> (none)
- D1: value Inolux_IN-PI554FCH -> XL-5050RGBC-WS2812B; LCSC Part # (none) -> C2843785
- D2: LCSC Part # (none) -> C191023
- E1: value Antenna -> ANT_CA-C03; Availability In Stock -> (none); Check_prices https://www.snapeda.com/parts/YC0010AA/Quectel/view-part/?r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 -> (none); LCSC Part # (none) -> C9900003739; MANUFACTURER Quectel -> (none); MAXIMUM_PACKAGE_HEIGHT 1.3 mm -> (none); MF Quectel -> (none); MP YC0010AA -> (none); PARTREV 1.1 -> (none); Package None -> (none); Price None -> (none); Purchase-URL https://www.snapeda.com/api/url_track_click_mouser/?unipart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 -> (none); STANDARD Manufacturer Recommendations -> (none); SnapEDA_Link https://www.snapeda.com/parts/YC0010AA/Quectel/view-part/?r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 -> (none)
- J1: LCSC Part # (none) -> C9900016956
- J2: now left out of the parts list
- Q1: value BC847B -> BC847BS; LCSC Part # (none) -> C8653
- Q2: LCSC Part # (none) -> C7202986
- S1: value TL3365AF180QG -> UK-B0267-SP25Y; Availability In Stock -> (none); Check_prices https://www.snapeda.com/parts/TL3365AF180QG/E-Switch/view-p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 -> (none); LCSC Part # (none) -> C493283; MANUFACTURER E-Switch -> (none); MAXIMUM_PACKAGE_HEIGHT 2.5 mm -> (none); MF E-Switch -> (none); MP TL3365AF180QG -> (none); PARTREV A -> (none); Package None -> (none); Price None -> (none); Purchase-URL https://www.snapeda.com/api/url_track_click_mouser/?unipart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 -> (none); SNAPEDA_PN TL3365AF180QG -> (none); STANDARD Manufacturer Recommendations -> (none); SnapEDA_Link https://www.snapeda.com/parts/TL3365AF180QG/E-Switch/view-p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 -> (none)
- S2: value TL3365AF180QG -> UK-B0267-SP25Y; Availability In Stock -> (none); Check_prices https://www.snapeda.com/parts/TL3365AF180QG/E-Switch/view-p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 -> (none); MANUFACTURER E-Switch -> (none); MAXIMUM_PACKAGE_HEIGHT 2.5 mm -> (none); MF E-Switch -> (none); MP TL3365AF180QG -> (none); PARTREV A -> (none); Package None -> (none); Price None -> (none); Purchase-URL https://www.snapeda.com/api/url_track_click_mouser/?unipart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 -> (none); SNAPEDA_PN TL3365AF180QG -> (none); STANDARD Manufacturer Recommendations -> (none); SnapEDA_Link https://www.snapeda.com/parts/TL3365AF180QG/E-Switch/view-p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 -> (none)
- U1: LCSC Part # (none) -> C2832759
- U2: LCSC Part # (none) -> C83291
- U3: LCSC Part # (none) -> C2846043
- U4: value TLV70233_SOT23-5 -> ME6211C33M5G-N; LCSC Part # (none) -> C82942
- U5: value MCP73831-2-OT -> MCP73831T-2ATI/OT; LCSC Part # (none) -> C14879
- U6: value LSM6DS3 -> LSM6DS3TR; LCSC Part # (none) -> C95230
Other:
- moved on the sheet: R7, R8

Commit message: update kicad
Parts:
- removed R10, R9: 0, Resistor_SMD:R_0603_1608Metric, symbol Device:R
Connections:
- net SCL is gone; now on net IO22_SCL: R7.1, U2.4 (SCK), U6.13 (SCL)
- net SDA is gone; now on net IO21_SDA: R8.1, U2.3 (SDI), U6.14 (SDA)
- net IO21 renamed IO21_SDA
- net IO22 renamed IO22_SCL
Changed lines of the file:
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@@
-    (stroke (width 0) (type default))
-  )
-  (wire (pts (xy 89.154 160.782) (xy 89.154 164.592))
     (stroke (width 0) (type default))
   )
@@
     (stroke (width 0) (type default))
   )
-  (wire (pts (xy 94.996 160.782) (xy 94.996 162.052))
-    (stroke (width 0) (type default))
-  )
   (wire (pts (xy 71.628 107.696) (xy 69.088 110.236))
     (stroke (width 0) (type default))
@@
     (stroke (width 0) (type default))
   )
-  (wire (pts (xy 94.996 162.052) (xy 101.6 162.052))
+  (wire (pts (xy 89.154 162.052) (xy 101.6 162.052))
     (stroke (width 0) (type default))
   )
@@
   )
   (wire (pts (xy 114.3 174.752) (xy 114.3 181.864))
-    (stroke (width 0) (type default))
-  )
-  (wire (pts (xy 94.996 151.13) (xy 94.996 153.162))
     (stroke (width 0) (type default))
   )
@@
     (stroke (width 0) (type default))
   )
-  (wire (pts (xy 89.154 151.13) (xy 89.154 153.162))
-    (stroke (width 0) (type default))
-  )
   (wire (pts (xy 145.288 167.894) (xy 142.748 167.894))
     (stroke (width 0) (type default))
@@
     (effects (font (size 1.27 1.27)) (justify left bottom))
   )
-  (label "SDA" (at 95.504 164.592 0) (fields_autoplaced)
-    (effects (font (size 1.27 1.27)) (justify left bottom))
-  )
-  (label "SCL" (at 37.592 170.688 0) (fields_autoplaced)
-    (effects (font (size 1.27 1.27)) (justify left bottom))
-  )
   (label "D-" (at 48.26 43.18 0) (fields_autoplaced)
     (effects (font (size 1.27 1.27)) (justify left bottom))
@@
     (effects (font (size 1.27 1.27)) (justify left bottom))
   )
-  (label "IO22" (at 260.858 101.6 0) (fields_autoplaced)
-    (effects (font (size 1.27 1.27)) (justify left bottom))
-  )
   (label "RX" (at 44.45 109.22 0) (fields_autoplaced)
     (effects (font (size 1.27 1.27)) (justify left bottom))
@@
     (effects (font (size 1.27 1.27)) (justify left bottom))
   )
+  (label "IO22_SCL" (at 37.592 170.688 0) (fields_autoplaced)
+    (effects (font (size 1.27 1.27)) (justify left bottom))
+  )
   (label "IO0" (at 145.542 104.902 0) (fields_autoplaced)
     (effects (font (size 1.27 1.27)) (justify left bottom))
@@
     (effects (font (size 1.27 1.27)) (justify left bottom))
   )
-  (label "SDA" (at 37.592 168.148 0) (fields_autoplaced)
-    (effects (font (size 1.27 1.27)) (justify left bottom))
-  )
-  (label "IO21" (at 89.154 151.13 0) (fields_autoplaced)
+  (label "IO21_SDA" (at 89.154 164.592 0) (fields_autoplaced)
+    (effects (font (size 1.27 1.27)) (justify left bottom))
+  )
+  (label "IO21_SDA" (at 37.592 168.148 0) (fields_autoplaced)
     (effects (font (size 1.27 1.27)) (justify left bottom))
   )
@@
     (effects (font (size 1.27 1.27)) (justify left bottom))
   )
-  (label "IO21" (at 260.858 99.06 0) (fields_autoplaced)
-    (effects (font (size 1.27 1.27)) (justify left bottom))
-  )
   (label "SDA1" (at 182.118 154.178 0) (fields_autoplaced)
     (effects (font (size 1.27 1.27)) (justify left bottom))
@@
     (effects (font (size 1.27 1.27)) (justify left bottom))
   )
+  (label "IO21_SDA" (at 260.858 99.06 0) (fields_autoplaced)
+    (effects (font (size 1.27 1.27)) (justify left bottom))
+  )
   (label "D+" (at 48.26 48.26 0) (fields_autoplaced)
     (effects (font (size 1.27 1.27)) (justify left bottom))
   )
-  (label "SCL" (at 94.996 162.052 0) (fields_autoplaced)
-    (effects (font (size 1.27 1.27)) (justify left bottom))
-  )
   (label "IO25" (at 260.858 106.68 0) (fields_autoplaced)
     (effects (font (size 1.27 1.27)) (justify left bottom))
@@
     (effects (font (size 1.27 1.27)) (justify left bottom))
   )
-  (label "IO22" (at 94.996 151.13 0) (fields_autoplaced)
+  (label "IO22_SCL" (at 89.154 162.052 0) (fields_autoplaced)
     (effects (font (size 1.27 1.27)) (justify left bottom))
   )
   (label "IO14" (at 260.604 88.9 0) (fields_autoplaced)
+    (effects (font (size 1.27 1.27)) (justify left bottom))
+  )
+  (label "IO22_SCL" (at 260.858 101.6 0) (fields_autoplaced)
     (effects (font (size 1.27 1.27)) (justify left bottom))
   )
@@
     )
   )
-  (symbol (lib_id "Device:R") (at 94.996 156.972 180) (unit 1)
-    (in_bom yes) (on_board yes) (dnp no)
-    (property "Reference" "R10" (at 92.456 156.972 90)
-      (effects (font (size 1.27 1.27)))
-    )
-    (property "Value" "0" (at 94.996 156.972 90)
-      (effects (font (size 1.27 1.27)))
-    )
-    (property "Footprint" "Resistor_SMD:R_0603_1608Metric" (at 96.774 156.972 90)
-      (effects (font (size 1.27 1.27)) hide)
-    )
-    (property "Datasheet" "~" (at 94.996 156.972 0)
-      (effects (font (size 1.27 1.27)) hide)
-    )
-    (pin "1")
-    (pin "2")
-    (instances
-      (project "OpenWear"
-        (path "/f2530224-e9e1-4854-8a1f-b76a7a8a2a4d"
-          (reference "R10") (unit 1)
-        )
-      )
-    )
-  )
   (symbol (lib_id "Transistor_BJT:BC847BDW1") (at 86.106 116.332 0) (mirror x) (unit 2)
     (in_bom yes) (on_board yes) (dnp no) (fields_autoplaced)
@@
         )
       )
-    )
-  )
-  (symbol (lib_id "Device:R") (at 89.154 156.972 180) (unit 1)
-    (in_bom yes) (on_board yes) (dnp no)
-    (property "Reference" "R9" (at 86.614 156.972 90)
-      (effects (font (size 1.27 1.27)))
-    )
-    (property "Value" "0" (at 89.154 156.972 90)
-      (effects (font (size 1.27 1.27)))
-    )
-    (property "Footprint" "Resistor_SMD:R_0603_1608Metric" (at 90.932 156.972 90)
-      (effects (font (size 1.27 1.27)) hide)
-    )
-    (property "Datasheet" "~" (at 89.154 156.972 0)
-      (effects (font (size 1.27 1.27)) hide)
-    )
-    (pin "1")
-    (pin "2")
-    (instances
-      (project "OpenWear"
-        (path "/f2530224-e9e1-4854-8a1f-b76a7a8a2a4d"
-          (reference "R9") (unit 1)
-        )
-      )
