File: Hardware/Kicad File/OpenWear.kicad_sch (KiCad schematic)
At the start: 39 parts, among them J1 USB_C, J2 Connector, Q1 BC847BS, Q2 DMG3415U, U1 ESP32-PICO-D4, U2 BMP280, U3 CH343P, U4 ME6211C33M5G-N, U5 MCP73831T-2ATI/OT, U6 LSM6DS3TR

Commit message: update pcb and sch
Parts:
- added C15: 4.7uF, Capacitor_SMD:C_0603_1608Metric, symbol Device:C
- C3: value 100nF -> 4.7uF
- R1: value 10K -> 1K
Connections:
- net +3.3V is gone; now on net +3V3: R5.1
- net +5V: now also C3.1, J2.14 (5V)
- net +BATT: now also C15.2; no longer C3.2, R2.1
- net DTR: now also U3.12 (DTR)
- net GND: now also C3.2, R2.1, C15.1; no longer C3.1
- net RTS: now also U3.13 (RTS)
- net VCC: no longer J2.14 (5V)
Other:
- note added: "200mA"
- moved on the sheet: C3

Commit message: update pcb and sch
Parts:
- added C16: 100nF, Capacitor_SMD:C_0603_1608Metric, symbol Device:C
Connections:
- net +3V3: now also U3.9 (VBUS), C16.1
- net GND: now also C16.2
- no-connect marks 33 -> 32
Other:
- moved on the sheet: C8, C9

Commit message: update sch
Connections:
- net VBUS: now also C3.1, Q2.1 (G), R1.2, U5.4 (V_{DD})
- net VCC: now also D2.1 (K), J2.14 (5V)
- removed net +5V: C3.1, D2.1 (K), J2.14 (5V), Q2.1 (G), R1.2, U5.4 (V_{DD})
Other:
- moved on the sheet: Q2
